Commit message: Adjust base_link origin position in mecanum.xacro

File: simulations/mentorpi_description/urdf/mecanum.xacro (robot description, xacro)
@@ -15,5 +15,5 @@
     <parent link="base_footprint"/>
     <child link="base_link"/>
-    <origin xyz="0 0 0.07" rpy="0 0 0"/>
+    <origin xyz="0 0 0.05" rpy="0 0 0"/>
   </joint>
   <link name="base_link">
